Commit message: fixed grasping task function

File: kuka_iiwa_support/urdf/kuka_iiwa_macro_ctrl_gripper.xacro (robot description, xacro)
@@ -235,5 +235,5 @@
       <parent link="${robot_name}_link_6"/>
       <child link="${robot_name}_link_7"/>
-      <origin xyz="0 0.081 0.06070" rpy="${- PI / 2} ${PI} 0"/>
+      <origin xyz="0 0.081 0.06070" rpy="${-PI/2} ${PI} 0"/>
       <axis xyz="0 0 1"/>
       <limit lower="${-175 * PI / 180}" upper="${175 * PI / 180}"
@@ -270,5 +270,5 @@
     <xacro:include filename="$(find wsg50_simulation)/urdf/wsg_50.urdf.xacro"/>
     <xacro:wsg_50_xacro name="wsg_50" parent="${robot_name}_link_ee">
-      <origin xyz="0 0 0" rpy="0 -${PI/2} 0"/>
+      <origin xyz="0 0 0" rpy="0 0 0"/>
     </xacro:wsg_50_xacro>
     <link name="${robot_name}_gripper_midpoint"></link>
@@ -276,5 +276,5 @@
       <parent link="wsg_50_base_link"/>
       <child link="${robot_name}_gripper_midpoint"/>
-      <origin xyz="0 0 0.15" rpy="0 0 0"/>
+      <origin xyz="0 0 0.15" rpy="0 0 1.57"/>
     </joint>
 		<xacro:transmission_block joint_name="${robot_name}_joint_1"/>

File: kuka_iiwa_support/urdf/kuka_iiwa_macro_vel_ctrl_gripper.xacro (robot description, xacro)
@@ -275,7 +275,7 @@
     <link name="${robot_name}_gripper_midpoint"></link>
     <joint name="${robot_name}_grasp_joint" type="fixed">
-      <parent link="wsg_50_base_link"/>
+      <parent link="${robot_name}_link_ee"/>
       <child link="${robot_name}_gripper_midpoint"/>
-      <origin xyz="0 0 0.15" rpy="0 0 0"/>
+      <origin xyz="0 0 0.15" rpy="0 0 ${PI/2}"/>
     </joint>
 		<xacro:transmission_block joint_name="${robot_name}_joint_1"/>
