Commit message: first grasp demo

File: kuka_iiwa_support/urdf/kuka_iiwa_macro_vel_ctrl_gripper.xacro (robot description, xacro)
@@ -273,9 +273,17 @@
       <origin xyz="0 0 0" rpy="0 -${PI/2} 0"/>
     </xacro:wsg_50_xacro>
-    <link name="${robot_name}_gripper_midpoint"></link>
+    <link name="${robot_name}_gripper_midpoint">
+    </link>
     <joint name="${robot_name}_grasp_joint" type="fixed">
       <parent link="${robot_name}_link_ee"/>
       <child link="${robot_name}_gripper_midpoint"/>
       <origin xyz="0 0 0.15" rpy="0 0 ${PI/2}"/>
+    </joint>
+    <link name="${robot_name}_plate_center">
+    </link>
+    <joint name="${robot_name}_plate_joint" type="fixed">
+      <parent link="${robot_name}_gripper_midpoint"/>
+      <child link="${robot_name}_plate_center"/>
+      <origin xyz="0 0 0.2" rpy="0 0 0"/>
     </joint>
 		<xacro:transmission_block joint_name="${robot_name}_joint_1"/>

Commit message: avoid plate added

File: kuka_iiwa_support/urdf/kuka_iiwa_macro_vel_ctrl_gripper.xacro (robot description, xacro)
@@ -278,5 +278,5 @@
       <parent link="${robot_name}_link_ee"/>
       <child link="${robot_name}_gripper_midpoint"/>
-      <origin xyz="0 0 0.15" rpy="0 0 ${PI/2}"/>
+      <origin xyz="0 0 0.14" rpy="0 0 ${PI/2}"/>
     </joint>
     <link name="${robot_name}_plate_center">
